File: G11_EMB_PCB1/G11_EMB_PCB1.kicad_pcb (KiCad board)
At the start: 2 copper layers, 95 x 75 mm, 5 parts, among them U1 SY8089AAAC

Commit message: 2024-10-03 M
Parts:
- added C2: 22u, Capacitor_SMD:C_0603_1608Metric_Pad1.08x0.95mm_HandSolder, F.Cu at (88.1, 64.5)
- added C3: 22u, Capacitor_SMD:C_0603_1608Metric_Pad1.08x0.95mm_HandSolder, F.Cu at (88.0, 62.0)
- added C5: 22u, Capacitor_SMD:C_0603_1608Metric_Pad1.08x0.95mm_HandSolder, F.Cu at (96.0, 66.5)
- added J1: Conn_01x01_MountingPin, Connector_PinHeader_2.54mm:PinHeader_1x01_P2.54mm_Vertical, F.Cu at (78.0, 66.5)
- added J2: Conn_01x01_MountingPin, Connector_PinHeader_2.54mm:PinHeader_1x01_P2.54mm_Vertical, F.Cu at (78.0, 75.5)
- added J3: Conn_01x01_MountingPin, Connector_PinHeader_2.54mm:PinHeader_1x01_P2.54mm_Vertical, F.Cu at (103.0, 76.0)
- added J4: Conn_01x01_MountingPin, Connector_PinHeader_2.54mm:PinHeader_1x01_P2.54mm_Vertical, F.Cu at (103.0, 66.5)
- added R1: R, Resistor_SMD:R_0603_1608Metric_Pad0.98x0.95mm_HandSolder, F.Cu at (87.9, 72.0)
- added R2: R, Resistor_SMD:R_0603_1608Metric_Pad0.98x0.95mm_HandSolder, F.Cu at (88.1, 74.0)
- added REF**: MountingHole_3.2mm_M3_Pad_Via, MountingHole:MountingHole_3.2mm_M3_Pad_Via, F.Cu at (55.0, 120.0)
- added REF**: MountingHole_3.2mm_M3_Pad_Via, MountingHole:MountingHole_3.2mm_M3_Pad_Via, F.Cu at (140.0, 55.0)
- added REF**: MountingHole_3.2mm_M3_Pad_Via, MountingHole:MountingHole_3.2mm_M3_Pad_Via, F.Cu at (55.0, 55.0)
- added REF**: MountingHole_3.2mm_M3_Pad_Via, MountingHole:MountingHole_3.2mm_M3_Pad_Via, F.Cu at (140.0, 120.0)
- moved L1 20.4 mm to (98.8, 71.0)
- moved C1 15.2 mm to (88.1, 67.0)
- moved C4 8.28 mm to (88.0, 76.0)
- moved U1 4.56 mm to (93.3, 71.0), turned to 180 degrees
- moved D1 4.38 mm to (82.5, 67.0), turned to 180 degrees
Routing:
- net (no net): vias 4 -> 0

Commit message: 2024-10-03
Parts:
- moved C3 41.2 mm to (95.6, 102.5)
- moved C2 40.2 mm to (95.6, 104.0)
- moved R1 39.3 mm to (95.6, 110.5)
- moved C1 39.2 mm to (95.6, 105.5)
- moved C5 39.2 mm to (103.5, 105.0)
- moved R2 38.7 mm to (95.6, 112.0)
- moved J1 38.3 mm to (86.0, 104.0)
- moved J2 38.3 mm to (86.0, 113.0)
- moved C4 38.3 mm to (95.6, 113.5)
- moved J4 38.2 mm to (110.5, 104.0)
- moved L1 38.2 mm to (106.3, 108.5)
- moved U1 38.2 mm to (100.8, 108.5)
- moved D1 37.9 mm to (91.0, 104.0)
- moved J3 37.8 mm to (110.5, 113.0)
Routing:
- net VIN: track 0.00 -> 3.90 mm
Other:
- board text added: "3.3V OUT"
- board text added: "5V IN"
- board text added: "GND"
- board text added: "SY8089"
- board text added: "TUES G11 EMB PCB1 PSU Demo board"

Commit message: 2024-10-04
Parts:
- added D2: LED, LED_SMD:LED_0603_1608Metric_Pad1.05x0.95mm_HandSolder, F.Cu at (103.2, 102.5)
- added R3: 220, Resistor_SMD:R_0603_1608Metric_Pad0.98x0.95mm_HandSolder, F.Cu at (107.0, 102.5)
- R1: value R -> 220k / 1%
- R2: value R -> 49.9k / 1%
- moved C4 4.20 mm to (96.5, 109.4)
- moved C1 2.86 mm to (98.5, 105.5)
- moved C2 2.86 mm to (98.5, 104.0)
- moved C3 2.86 mm to (98.5, 102.5)
- moved D1 2.10 mm to (93.0, 104.0)
- moved J2 2.09 mm to (88.0, 112.4)
- moved J1 2.00 mm to (88.0, 104.0)
- moved R1 1.00 mm to (96.5, 110.9)
- moved R2 1.00 mm to (96.5, 112.4), turned to 180 degrees
- moved J3 0.78 mm to (111.0, 112.4)
- moved C5 0.60 mm to (103.2, 105.5)
- moved J4 0.50 mm to (111.0, 104.0)
- moved L1 0.40 mm to (106.3, 108.9)
Routing:
- net VCC_SY: track 0.00 -> 30.3 mm, vias 0 -> 3
- net Net-(D1-K): track 0.00 -> 18.3 mm, vias 0 -> 2
- net Net-(U1-FB): track 0.00 -> 5.14 mm
- net Net-(U1-LX): track 0.00 -> 5.00 mm
- net Net-(D2-A): track 0.00 -> 2.05 mm
- added copper zone on B.Cu, net GND
- added copper zone on F.Cu, net GND
- added copper zone on F.Cu, net Net-(U1-LX)
Other:
- board text added: "SY8089AAAC"
- board text removed: "SY8089"
