File: G11_EMB_PCB1/SY8089AAAC.kicad_sch (KiCad schematic)
At the start: 10 parts, among them U1 SY8089AAAC

Commit message: 2024-10-02
Parts:
- C1, C4: footprint (none) -> Capacitor_SMD:C_0603_1608Metric_Pad1.08x0.95mm_HandSolder
- L1: footprint (none) -> Inductor_SMD:L_Coilcraft_XxL4020
- U1: footprint (none) -> Package_TO_SOT_SMD:SOT-23-5_HandSoldering
Changed lines of the file:
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@@
 			)
 		)
-		(property "Footprint" ""
+		(property "Footprint" "Inductor_SMD:L_Coilcraft_XxL4020"
 			(at 160.02 88.9 0)
 			(effects
@@
 			)
 		)
-		(property "Footprint" ""
+		(property "Footprint" "Capacitor_SMD:C_0603_1608Metric_Pad1.08x0.95mm_HandSolder"
 			(at 114.3 97.79 0)
 			(effects
@@
 			)
 		)
-		(property "Footprint" ""
+		(property "Footprint" "Capacitor_SMD:C_0603_1608Metric_Pad1.08x0.95mm_HandSolder"
 			(at 166.37 97.79 0)
 			(effects
@@
 			)
 		)
-		(property "Footprint" ""
+		(property "Footprint" "Package_TO_SOT_SMD:SOT-23-5_HandSoldering"
 			(at 148.082 87.63 0)
 			(effects

Commit message: 2024-10-03 M
Parts:
- added J1, J2, J3, J4: Conn_01x01_MountingPin, PinHeader_1x01_P2.54mm_Vertical, symbol Connector_Generic_MountingPin:Conn_01x01_MountingPin
- C2, C3, C5: footprint (none) -> Capacitor_SMD:C_0603_1608Metric_Pad1.08x0.95mm_HandSolder
- R1, R2: footprint (none) -> Resistor_SMD:R_0603_1608Metric_Pad0.98x0.95mm_HandSolder
Connections:
- net GND: now also J2.1 (Pin_1), J3.1 (Pin_1)
- net VCC_SY: now also J4.1 (Pin_1)
- net VIN: now also J1.1 (Pin_1)

Commit message: 2024-10-04
Parts:
- added D2: LED, LED_SMD:LED_0603_1608Metric_Pad1.05x0.95mm_HandSolder, symbol Device:LED
- added R3: 220, Resistor_SMD:R_0603_1608Metric_Pad0.98x0.95mm_HandSolder, symbol Device:R
- R1: value R -> 220k / 1%
- R2: value R -> 49.9k / 1%
Connections:
- net GND: now also D2.1 (K)
- net VCC_SY: now also R3.1
- new net: D2.2 (A), R3.2
